File: board/A500r5_eprom_adapter/A500r5_eprom_adapter-plcc32-invert.kicad_pcb (KiCad board)
At the start: 2 copper layers, 40.6 x 54.6 mm, 9 parts, among them J2 A18 Selector, J3 A19 Selector, U1 27C400-A500, U2 27C080-L, U3 27C080-L

Commit message: More gerbers
Other:
- board text added: "A500 rev.5 27C0x0 ROM Adapter"
- board text added: "tabaglio@posteo.net"
Changed lines of the file:
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@@
   (general
     (thickness 1.6)
-    (drawings 13)
+    (drawings 15)
     (tracks 731)
     (zones 0)
@@
     )
   )
+  (gr_text tabaglio@posteo.net (at 116.84 124.46) (layer F.SilkS)
+    (effects (font (size 1 1) (thickness 0.15) italic))
+  )
+  (gr_text "A500 rev.5\n27C0x0 ROM Adapter" (at 118.11 101.6 90) (layer F.SilkS)
+    (effects (font (size 2 2) (thickness 0.15)))
+  )
   (gr_text A19 (at 138.43 102.87) (layer F.SilkS)
     (effects (font (size 1 1) (thickness 0.15)))
@@
     (effects (font (size 1 1) (thickness 0.15)))
   )
-  (gr_text HIGH (at 138.43 123.19) (layer B.SilkS)
-    (effects (font (size 1 1) (thickness 0.15)) (justify mirror))
+  (gr_text HIGH (at 138.43 123.19) (layer F.SilkS)
+    (effects (font (size 1 1) (thickness 0.15)))
   )
   (gr_text 27C040/27C080 (at 146.05 99.06 90) (layer F.SilkS)
