File: board/A500r5_eprom_adapter-DIP/A500r5_eprom_adapter.kicad_pcb (KiCad board)
At the start: 2 copper layers, 39.4 x 86.4 mm, 11 parts, among them J2 A18 Selector, J3 A19 Selector, U1 27C400-A500, U2 27C080-L, U3 27C080-L

Commit message: Draw rev.2 DIP PCB
Parts:
- added J4: A17 Selection, Connector_PinHeader_2.54mm:PinHeader_1x03_P2.54mm_Vertical, F.Cu at (116.8, 57.1)
Connections:
- U1 pad 1: (no net) -> /SOCK_P1
- U1 pad 31: /A17 -> /SOCK_P31
Routing:
- net /SOCK_P31: track 0.00 -> 71.4 mm
- net /A13: track 69.2 -> 138.9 mm
- net /D7-H: track 105.8 -> 45.5 mm, vias 1 -> 2
- net /A17: track 68.3 -> 117.0 mm
- net /SOCK_P1: track 0.00 -> 19.9 mm
- net /A8: track 117.2 -> 98.7 mm, vias 0 -> 2
- net /A7: track 82.1 -> 64.5 mm, vias 0 -> 2
- net /~OE: track 92.8 -> 109.3 mm
- net /A4: track 77.1 -> 67.6 mm
- net /A5: track 67.9 -> 77.0 mm
- net /D6-H: track 37.0 -> 45.6 mm
- net GND: track 122.4 -> 130.6 mm, vias 0 -> 1
- net /A3: track 68.5 -> 75.9 mm, vias 0 -> 2
- net /A0: track 74.2 -> 67.0 mm, vias 1 -> 0
- net /A16: track 57.9 -> 51.2 mm, vias 1 -> 0
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Other:
- board text added: "J4: 1-2 -> A17 on PIN1 2-3 -> A17 on PIN31"
- board text added: "Rev. 2"

Commit message: Add rev.2 boards
Other:
- board text removed: "rev.1"
